Commit message: add left front and back arms

File: forg_description/urdf/back_arm.urdf.xacro (robot description, xacro)
@@ -2,17 +2,18 @@
 <robot xmlns:xacro="http://www.ros.org/wiki/xacro">
   <xacro:include filename="inertial_macros.urdf.xacro"/>
-  <xacro:include filename="wheel.urdf.xacro"/>
 	<xacro:arg name="ignition" default="false"/>
-	<xacro:macro name="wheel_steering" params="name parent *origin **mirror">
-    <joint name="${name}_base_joint" type="fixed">
+	<xacro:macro name="back_arm" params="name parent *origin **mirror">
+    <joint name="${name}_joint" type="continuous">
 			<parent link="${parent}"/>
 			<child link="${name}"/>
       <xacro:insert_block name="origin"/>
+			<axis xyz="1 0 0"/>
 		</joint>
-    <link name="${name}_base">
+    <link name="${name}">
 			<visual>
+        <origin xyz="0 0 0"/>
 				<xacro:insert_block name="mirror"/>
 				<geometry>
-					<mesh filename="package://forg_description/meshes/steering_base.dae"/>
+					<mesh filename="package://forg_description/meshes/back_arm.dae"/>
 				</geometry>
 			</visual>
@@ -21,5 +22,5 @@
         <xacro:insert_block name="mirror"/>
 				<geometry>
-					<mesh filename="package://forg_description/meshes/steering_base.dae"/>
+					<mesh filename="package://forg_description/meshes/back_arm.dae"/>
 				</geometry>
 			</collision>
@@ -29,10 +30,4 @@
       </xacro:inertial_box>
 		</link>
-    <xacro:wheel name="${name}" parent="${name}_base">
-    <origin xyz="0 ${0.15+0.045+0.11-0.035} ${0.03-0.5}" rpy="${pi/2} 0 ${-pi}"/>
-    <mirror>
-      <origin rpy="0 0 0"/>
-    </mirror>
-  </xacro:wheel>
 	</xacro:macro>
 </robot>

File: forg_description/urdf/forg_core.urdf.xacro (robot description, xacro)
@@ -4,4 +4,6 @@
   <xacro:include filename="base.urdf.xacro"/>
   <xacro:include filename="middle_arm.urdf.xacro"/>
+  <xacro:include filename="front_arm.urdf.xacro"/>
+  <xacro:include filename="back_arm.urdf.xacro"/>
   <link name="base_footprint"/>
   <joint name="base_footprint_to_base_link_joint" type="fixed">
@@ -24,5 +26,11 @@
     </mirror>
   </xacro:middle_arm>
-  <xacro:wheel name="front_left_wheel" parent="left_middle_arm">
+  <xacro:front_arm name="left_front_arm" parent="left_middle_arm">
+    <origin xyz="${0.11/2 + 0.045/2} 0 0" rpy="0 0 0"/>
+    <mirror>
+      <origin rpy="0 0 0"/>
+    </mirror>
+  </xacro:front_arm>
+  <xacro:wheel name="left_front_wheel_steering" parent="left_front_arm">
     <origin xyz="${0.15+0.045+0.11-0.035} -0.2 ${0.03-0.5}" rpy="0 ${pi/2} 0"/>
     <mirror>
@@ -30,6 +38,18 @@
     </mirror>
   </xacro:wheel>
+  <xacro:wheel name="left_front_wheel" parent="left_middle_arm">
+    <origin xyz="${0.15+0.045+0.11-0.035} -0.2 ${0.03-0.5}" rpy="0 ${pi/2} 0"/>
+    <mirror>
+      <origin rpy="0 0 0"/>
+    </mirror>
+  </xacro:wheel>
+  <xacro:back_arm name="left_back_arm" parent="left_middle_arm">
+    <origin xyz="${0.045/2 + 0.11 - 0.07/2} ${0.18 + 0.2} ${-0.075}" rpy="0 0 0"/>
+    <mirror>
+      <origin rpy="0 0 0"/>
+    </mirror>
+  </xacro:back_arm>
   <xacro:middle_arm name="right_middle_arm" parent="base">
-    <origin xyz="${-0.255/2 - 0.05} ${0.045-0.225} 0" rpy="0 ${pi/2} 0"/>
+    <origin xyz="${-0.255/2 - 0.05} ${0.045-0.225} 0" rpy="${pi} ${pi/2} 0"/>
     <mirror>
       <origin rpy="0 0 ${pi}"/>

File: forg_description/urdf/front_arm.urdf.xacro (robot description, xacro)
@@ -2,37 +2,32 @@
 <robot xmlns:xacro="http://www.ros.org/wiki/xacro">
   <xacro:include filename="inertial_macros.urdf.xacro"/>
-  <xacro:include filename="wheel.urdf.xacro"/>
 	<xacro:arg name="ignition" default="false"/>
-	<xacro:macro name="wheel_steering" params="name parent *origin **mirror">
-    <joint name="${name}_base_joint" type="fixed">
+	<xacro:macro name="front_arm" params="name parent *origin **mirror">
+    <joint name="${name}_joint" type="continuous">
 			<parent link="${parent}"/>
 			<child link="${name}"/>
       <xacro:insert_block name="origin"/>
+			<axis xyz="1 0 0"/>
 		</joint>
-    <link name="${name}_base">
+    <link name="${name}">
 			<visual>
+        <origin xyz="0 ${-0.07-0.18-0.015} ${-0.15 - 0.09/2}"/>
 				<xacro:insert_block name="mirror"/>
 				<geometry>
-					<mesh filename="package://forg_description/meshes/steering_base.dae"/>
+					<mesh filename="package://forg_description/meshes/front_arm.dae"/>
 				</geometry>
 			</visual>
 			<collision>
-        <origin xyz="0 0 0"/>
+        <origin xyz="0 ${-0.07-0.18-0.015} ${-0.15 - 0.09/2}"/>
         <xacro:insert_block name="mirror"/>
 				<geometry>
-					<mesh filename="package://forg_description/meshes/steering_base.dae"/>
+					<mesh filename="package://forg_description/meshes/front_arm.dae"/>
 				</geometry>
 			</collision>
       <xacro:inertial_box mass="0.05" x="0.17" y="0.00625" z="0.8"> <!-- TODO: replace shoulder axis mass with real value -->
-        <origin xyz="0 0 0"/>
+        <origin xyz="0 ${-0.07-0.18-0.015} ${-0.15 - 0.09/2}"/>
 				<xacro:insert_block name="mirror"/>
       </xacro:inertial_box>
 		</link>
-    <xacro:wheel name="${name}" parent="${name}_base">
-    <origin xyz="0 ${0.15+0.045+0.11-0.035} ${0.03-0.5}" rpy="${pi/2} 0 ${-pi}"/>
-    <mirror>
-      <origin rpy="0 0 0"/>
-    </mirror>
-  </xacro:wheel>
 	</xacro:macro>
 </robot>

File: forg_description/urdf/middle_arm.urdf.xacro (robot description, xacro)
@@ -8,5 +8,4 @@
 			<child link="${name}_shoulder_axis"/>
 			<xacro:insert_block name="origin"/>
-      <xacro:insert_block name="mirror"/>
 			<axis xyz="0 0 1"/>
 		</joint>
@@ -14,4 +13,5 @@
 			<visual>
 				<xacro:insert_block name="mirror"/>
+				<xacro:insert_block name="origin"/>
 				<geometry>
 					<mesh filename="package://forg_description/meshes/shoulder_axis.dae"/>
@@ -44,5 +44,4 @@
 			</visual>
 			<collision>
-        <xacro:insert_block name="origin"/>
         <xacro:insert_block name="mirror"/>
 				<geometry>
@@ -50,8 +49,8 @@
 				</geometry>
 			</collision>
-      <xacro:inertial_cylinder mass="0.05" length="0.17" radius="0.00625"> <!-- TODO: replace shoulder axis mass with real value -->
-				<xacro:insert_block name="origin"/>
+      <xacro:inertial_box mass="0.05" x="0.17" y="0.00625" z="0.8"> <!-- TODO: replace shoulder axis mass with real value -->
+        <origin xyz="0 0 0"/>
 				<xacro:insert_block name="mirror"/>
-      </xacro:inertial_cylinder>
+      </xacro:inertial_box>
 		</link>
 	</xacro:macro>
