Commit message: change kinematics computation
it works for vy = 0

File: forg_description/urdf/wheel_steering.urdf.xacro (robot description, xacro)
@@ -27,5 +27,5 @@
 			<child link="${name}_steering_gear"/>
       <origin xyz="0 0 ${0.15/2 - 0.005}"/>
-      <axis xyz="0 0 1"/>
+      <axis xyz="0 0 -1"/>
 		</joint>
     <link name="${name}_steering_gear">
