Commit message: delete mimic joint references

File: forg_description/urdf/forg_bot.urdf.xacro (robot description, xacro)
@@ -1,5 +1,5 @@
 <?xml version="1.0"?>
 <robot xmlns:xacro="http://www.ros.org/wiki/xacro" name="forg_bot">
-	<xacro:arg name="simulation" default="true"/>
+	<xacro:arg name="simulation" default="false"/>
   <xacro:include filename="forg_core.urdf.xacro"/>
   <xacro:include filename="ros2_control.urdf.xacro"/>

File: forg_description/urdf/forg_core.urdf.xacro (robot description, xacro)
@@ -5,5 +5,4 @@
   <xacro:include filename="left_front_arm.urdf.xacro"/>
   <xacro:include filename="left_back_arm.urdf.xacro"/>
-  <xacro:include filename="mimic_joint_plugin_macro.urdf.xacro"/>
   <xacro:include filename="right_middle_arm.urdf.xacro"/>
   <xacro:include filename="right_front_arm.urdf.xacro"/>
@@ -34,13 +33,12 @@
   </link>
   <joint name="shoulder_left_joint" type="continuous">
+    <mimic joint="shoulder_right_joint" multiplier="-1"/>
     <parent link="base"/>
     <child link="shoulder_left"/>
     <origin xyz="${0.255/2 + 0.05} ${0.045-0.225} 0"/>
     <axis xyz="1 0 0"/>
-    <mimic joint="shoulder_joint" multiplier="1"/>
     <limit effort="${10}" velocity="${360*2*pi/60}"/>
     <dynamics damping="0.1" friction="50"/> <!-- TODO replace with real properties -->
   </joint>
-  <!-- <xacro:mimic_joint_plugin_gazebo name_prefix="shoulder_left" parent_joint="shoulder_joint" mimic_joint="shoulder_left_joint" multiplier="1.0" /> -->
   <link name="shoulder_left">
   </link>
@@ -50,9 +48,7 @@
     <origin xyz="${-0.255/2 - 0.05} ${0.045-0.225} 0"/>
     <axis xyz="1 0 0"/>
-    <mimic joint="shoulder_joint" multiplier="-1"/>
     <limit effort="${10}" velocity="${360*2*pi/60}"/>
     <dynamics damping="0.1" friction="50"/> <!-- TODO replace with real properties -->
   </joint>
-  <xacro:mimic_joint_plugin_gazebo name_prefix="shoulder_right" parent_joint="shoulder_left_joint" mimic_joint="shoulder_right_joint" multiplier="-1.0" debug="false" use_pid="true" kp="100.0" ki="100.0" kd="100.0"/>
   <link name="shoulder_right">
   </link>

File: forg_description/urdf/wheel.urdf.xacro (robot description, xacro)
@@ -2,5 +2,4 @@
 <robot xmlns:xacro="http://www.ros.org/wiki/xacro">
   <xacro:include filename="inertial_macros.urdf.xacro"/>
-	<xacro:arg name="ignition" default="false"/>
 	<xacro:macro name="wheel" params="name parent *origin">
     <joint name="${name}_joint" type="continuous">

File: forg_description/urdf/wheel_steering.urdf.xacro (robot description, xacro)
@@ -3,5 +3,4 @@
   <xacro:include filename="inertial_macros.urdf.xacro"/>
   <xacro:include filename="wheel.urdf.xacro"/>
-	<xacro:arg name="ignition" default="false"/>
 	<xacro:macro name="wheel_steering" params="name parent *origin">
     <joint name="${name}_base_joint" type="fixed">
