Commit message: use wheel collision as sphere

File: forg_description/urdf/wheel.urdf.xacro (robot description, xacro)
@@ -39,5 +39,6 @@
 			<collision>
 				<geometry>
-					<mesh filename="package://forg_description/meshes/wheel.dae"/>
+					<!-- <mesh filename="package://forg_description/meshes/wheel.dae"/> -->
+          <sphere radius="0.06"/>
 				</geometry>
 			</collision>
