Commit message: add kinematics visualization for simulation

File: forg_description/urdf/ros2_control.urdf.xacro (robot description, xacro)
@@ -79,18 +79,24 @@
         <state_interface name="effort"/>
       </joint>
-      <!-- <joint name="shoulder_left_joint"> -->
-      <!--   <command_interface name="position"/> -->
-      <!--   <state_interface name="position"/> -->
-      <!--   <state_interface name="velocity"/> -->
-      <!--   <state_interface name="effort"/> -->
-      <!-- </joint> -->
-      <!-- <joint name="shoulder_right_joint"> -->
-      <!--   <param name="mimic">shoulder_left_joint</param> -->
-      <!--   <param name="multiplier">-1</param> -->
-      <!--   <command_interface name="position"/> -->
-      <!--   <state_interface name="position"/> -->
-      <!--   <state_interface name="velocity"/> -->
-      <!--   <state_interface name="effort"/> -->
-      <!-- </joint> -->
+      <joint name="shoulder_left_joint">
+        <state_interface name="position"/>
+        <state_interface name="velocity"/>
+        <state_interface name="effort"/>
+      </joint>
+      <joint name="shoulder_right_joint">
+        <state_interface name="position"/>
+        <state_interface name="velocity"/>
+        <state_interface name="effort"/>
+      </joint>
+      <joint name="left_back_arm_joint">
+        <state_interface name="position"/>
+        <state_interface name="velocity"/>
+        <state_interface name="effort"/>
+      </joint>
+      <joint name="right_back_arm_joint">
+        <state_interface name="position"/>
+        <state_interface name="velocity"/>
+        <state_interface name="effort"/>
+      </joint>
     </ros2_control>
     <gazebo>
