Commit message: insert xacros verbosely instead of trying to mirror meshes

File: forg_description/urdf/base.urdf.xacro (robot description, xacro)
@@ -3,5 +3,5 @@
   <xacro:include filename="inertial_macros.urdf.xacro"/>
 	<xacro:arg name="ignition" default="false"/>
-	<xacro:macro name="base" params="name parent *origin **mirror">
+	<xacro:macro name="base" params="name parent *origin">
     <joint name="${name}_joint" type="fixed">
 			<parent link="${parent}"/>
@@ -12,5 +12,4 @@
     <link name="${name}">
 			<visual>
-				<xacro:insert_block name="mirror"/>
 				<geometry>
 					<mesh filename="package://forg_description/meshes/spine.dae"/>
@@ -18,14 +17,9 @@
 			</visual>
 			<collision>
-        <xacro:insert_block name="origin"/>
-        <xacro:insert_block name="mirror"/>
 				<geometry>
 					<mesh filename="package://forg_description/meshes/spine.dae"/>
 				</geometry>
 			</collision>
-      <xacro:inertial_box mass="5" x="0.17" y="0.17" z="0.17"> <!-- TODO: replace with real values -->
-				<xacro:insert_block name="origin"/>
-				<xacro:insert_block name="mirror"/>
-      </xacro:inertial_box>
+      <xacro:inertial_box mass="5" x="0.17" y="0.17" z="0.17"/> <!-- TODO: replace with real values -->
 		</link>
 	</xacro:macro>

File: forg_description/urdf/forg_core.urdf.xacro (robot description, xacro)
@@ -1,9 +1,13 @@
 <?xml version="1.0" ?>
 <robot xmlns:xacro="http://www.ros.org/wiki/xacro">
+  <xacro:include filename="base.urdf.xacro"/>
+  <xacro:include filename="left_middle_arm.urdf.xacro"/>
+  <xacro:include filename="left_front_arm.urdf.xacro"/>
+  <xacro:include filename="left_back_arm.urdf.xacro"/>
+  <xacro:include filename="right_middle_arm.urdf.xacro"/>
+  <xacro:include filename="right_front_arm.urdf.xacro"/>
+  <xacro:include filename="right_back_arm.urdf.xacro"/>
+  <xacro:include filename="wheel_steering.urdf.xacro"/>
   <xacro:include filename="wheel.urdf.xacro"/>
-  <xacro:include filename="base.urdf.xacro"/>
-  <xacro:include filename="middle_arm.urdf.xacro"/>
-  <xacro:include filename="front_arm.urdf.xacro"/>
-  <xacro:include filename="back_arm.urdf.xacro"/>
   <link name="base_footprint"/>
   <joint name="base_footprint_to_base_link_joint" type="fixed">
@@ -15,44 +19,26 @@
   <link name="base_link"/>
   <xacro:base name="base" parent="base_link">
-    <origin xyz="0 0 0" rpy="0 0 ${pi/2}"/>
-    <mirror>
-      <origin rpy="0 0 0"/>
-    </mirror>
+    <origin xyz="0 0 0.5" rpy="0 0 ${pi/2}"/>
   </xacro:base>
-  <xacro:middle_arm name="left_middle_arm" parent="base">
+  <xacro:left_middle_arm name="left_middle_arm" parent="base">
     <origin xyz="${0.255/2 + 0.05} ${0.045-0.225} 0" rpy="0 ${pi/2} 0"/>
-    <mirror>
-      <origin rpy="0 0 0"/>
-    </mirror>
-  </xacro:middle_arm>
-  <xacro:front_arm name="left_front_arm" parent="left_middle_arm">
-    <origin xyz="${0.11/2 + 0.045/2} 0 0" rpy="0 0 0"/>
-    <mirror>
-      <origin rpy="0 0 0"/>
-    </mirror>
-  </xacro:front_arm>
-  <xacro:wheel name="left_front_wheel_steering" parent="left_front_arm">
-    <origin xyz="${0.15+0.045+0.11-0.035} -0.2 ${0.03-0.5}" rpy="0 ${pi/2} 0"/>
-    <mirror>
-      <origin rpy="0 0 0"/>
-    </mirror>
-  </xacro:wheel>
-  <xacro:wheel name="left_front_wheel" parent="left_middle_arm">
-    <origin xyz="${0.15+0.045+0.11-0.035} -0.2 ${0.03-0.5}" rpy="0 ${pi/2} 0"/>
-    <mirror>
-      <origin rpy="0 0 0"/>
-    </mirror>
-  </xacro:wheel>
-  <xacro:back_arm name="left_back_arm" parent="left_middle_arm">
+  </xacro:left_middle_arm>
+  <xacro:left_front_arm name="left_front_arm" parent="left_middle_arm">
+    <origin xyz="${0.045/2 + 0.11 - 0.07/2} 0 0" rpy="0 0 0"/>
+  </xacro:left_front_arm>
+  <xacro:wheel_steering name="left_front_wheel" parent="left_front_arm">
+    <origin xyz="0 ${-0.07-0.18-0.015} ${-0.15}" rpy="${pi} 0 0"/>
+  </xacro:wheel_steering>
+  <xacro:left_back_arm name="left_back_arm" parent="left_middle_arm">
     <origin xyz="${0.045/2 + 0.11 - 0.07/2} ${0.18 + 0.2} ${-0.075}" rpy="0 0 0"/>
-    <mirror>
-      <origin rpy="0 0 0"/>
-    </mirror>
-  </xacro:back_arm>
-  <xacro:middle_arm name="right_middle_arm" parent="base">
-    <origin xyz="${-0.255/2 - 0.05} ${0.045-0.225} 0" rpy="${pi} ${pi/2} 0"/>
-    <mirror>
-      <origin rpy="0 0 ${pi}"/>
-    </mirror>
-  </xacro:middle_arm>
+  </xacro:left_back_arm>
+  <xacro:right_middle_arm name="right_middle_arm" parent="base">
+    <origin xyz="${-0.255/2 - 0.05} ${0.045-0.225} 0" rpy="0 ${pi/2} 0"/>
+  </xacro:right_middle_arm>
+  <xacro:right_front_arm name="right_front_arm" parent="right_middle_arm">
+    <origin xyz="${-0.045/2 - 0.11 + 0.07/2} 0 0" rpy="0 0 0"/>
+  </xacro:right_front_arm>
+  <xacro:right_back_arm name="right_back_arm" parent="right_middle_arm">
+    <origin xyz="${-0.045/2 - 0.11 + 0.07/2} ${0.18 + 0.2} ${-0.075}" rpy="0 0 0"/>
+  </xacro:right_back_arm>
 </robot>

File: forg_description/urdf/inertial_macros.urdf.xacro (robot description, xacro)
@@ -3,8 +3,6 @@
     <!-- Specify some standard inertial calculations https://en.wikipedia.org/wiki/List_of_moments_of_inertia -->
     <!-- These make use of xacro's mathematical functionality -->
-    <xacro:macro name="inertial_sphere" params="mass radius *origin **mirror">
+    <xacro:macro name="inertial_sphere" params="mass radius">
         <inertial>
-				    <xacro:insert_block name="mirror"/>
-            <xacro:insert_block name="origin"/>
             <mass value="${mass}" />
             <inertia ixx="${(2/5) * mass * (radius*radius)}" ixy="0.0" ixz="0.0"
@@ -13,8 +11,6 @@
         </inertial>
     </xacro:macro>
-    <xacro:macro name="inertial_box" params="mass x y z *origin **mirror">
+    <xacro:macro name="inertial_box" params="mass x y z">
         <inertial>
-				    <xacro:insert_block name="mirror"/>
-            <xacro:insert_block name="origin"/>
             <mass value="${mass}" />
             <inertia ixx="${(1/12) * mass * (y*y+z*z)}" ixy="0.0" ixz="0.0"
@@ -23,8 +19,6 @@
         </inertial>
     </xacro:macro>
-    <xacro:macro name="inertial_cylinder" params="mass length radius *origin **mirror">
+    <xacro:macro name="inertial_cylinder" params="mass length radius">
         <inertial>
-				    <xacro:insert_block name="mirror"/>
-            <xacro:insert_block name="origin"/>
             <mass value="${mass}" />
             <inertia ixx="${(1/12) * mass * (3*radius*radius + length*length)}" ixy="0.0" ixz="0.0"

File: forg_description/urdf/left_front_arm.urdf.xacro (robot description, xacro)
@@ -3,5 +3,5 @@
   <xacro:include filename="inertial_macros.urdf.xacro"/>
 	<xacro:arg name="ignition" default="false"/>
-	<xacro:macro name="front_arm" params="name parent *origin **mirror">
+	<xacro:macro name="left_front_arm" params="name parent *origin">
     <joint name="${name}_joint" type="continuous">
 			<parent link="${parent}"/>
@@ -12,21 +12,14 @@
     <link name="${name}">
 			<visual>
-        <origin xyz="0 ${-0.07-0.18-0.015} ${-0.15 - 0.09/2}"/>
-				<xacro:insert_block name="mirror"/>
 				<geometry>
-					<mesh filename="package://forg_description/meshes/front_arm.dae"/>
+					<mesh filename="package://forg_description/meshes/left_front_arm.dae"/>
 				</geometry>
 			</visual>
 			<collision>
-        <origin xyz="0 ${-0.07-0.18-0.015} ${-0.15 - 0.09/2}"/>
-        <xacro:insert_block name="mirror"/>
 				<geometry>
-					<mesh filename="package://forg_description/meshes/front_arm.dae"/>
+					<mesh filename="package://forg_description/meshes/left_front_arm.dae"/>
 				</geometry>
 			</collision>
-      <xacro:inertial_box mass="0.05" x="0.17" y="0.00625" z="0.8"> <!-- TODO: replace shoulder axis mass with real value -->
-        <origin xyz="0 ${-0.07-0.18-0.015} ${-0.15 - 0.09/2}"/>
-				<xacro:insert_block name="mirror"/>
-      </xacro:inertial_box>
+      <xacro:inertial_box mass="0.05" x="0.17" y="0.00625" z="0.8"/> <!-- TODO: replace shoulder axis mass with real value -->
 		</link>
 	</xacro:macro>

File: forg_description/urdf/right_back_arm.urdf.xacro (robot description, xacro)
@@ -3,5 +3,5 @@
   <xacro:include filename="inertial_macros.urdf.xacro"/>
 	<xacro:arg name="ignition" default="false"/>
-	<xacro:macro name="left_back_arm" params="name parent *origin">
+	<xacro:macro name="right_back_arm" params="name parent *origin">
     <joint name="${name}_joint" type="continuous">
 			<parent link="${parent}"/>
@@ -13,10 +13,10 @@
 			<visual>
 				<geometry>
-					<mesh filename="package://forg_description/meshes/left_back_arm.dae"/>
+					<mesh filename="package://forg_description/meshes/right_back_arm.dae"/>
 				</geometry>
 			</visual>
 			<collision>
 				<geometry>
-					<mesh filename="package://forg_description/meshes/left_back_arm.dae"/>
+					<mesh filename="package://forg_description/meshes/right_back_arm.dae"/>
 				</geometry>
 			</collision>

File: forg_description/urdf/right_front_arm.urdf.xacro (robot description, xacro)
@@ -3,5 +3,5 @@
   <xacro:include filename="inertial_macros.urdf.xacro"/>
 	<xacro:arg name="ignition" default="false"/>
-	<xacro:macro name="left_back_arm" params="name parent *origin">
+	<xacro:macro name="right_front_arm" params="name parent *origin">
     <joint name="${name}_joint" type="continuous">
 			<parent link="${parent}"/>
@@ -13,10 +13,10 @@
 			<visual>
 				<geometry>
-					<mesh filename="package://forg_description/meshes/left_back_arm.dae"/>
+					<mesh filename="package://forg_description/meshes/right_front_arm.dae"/>
 				</geometry>
 			</visual>
 			<collision>
 				<geometry>
-					<mesh filename="package://forg_description/meshes/left_back_arm.dae"/>
+					<mesh filename="package://forg_description/meshes/right_front_arm.dae"/>
 				</geometry>
 			</collision>

File: forg_description/urdf/right_middle_arm.urdf.xacro (robot description, xacro)
@@ -3,5 +3,5 @@
   <xacro:include filename="inertial_macros.urdf.xacro"/>
 	<xacro:arg name="ignition" default="false"/>
-	<xacro:macro name="left_middle_arm" params="name parent *origin">
+	<xacro:macro name="right_middle_arm" params="name parent *origin">
     <joint name="${name}_shoulder_axis_joint" type="continuous">
 			<parent link="${parent}"/>
@@ -26,5 +26,5 @@
 			<parent link="${name}_shoulder_axis"/>
 			<child link="${name}"/>
-      <origin xyz="0 0 ${-0.005}" rpy="0 ${-pi/2} 0"/>
+      <origin xyz="0 0 ${0.005}" rpy="0 ${-pi/2} 0"/>
 			<axis xyz="0 0 1"/>
 		</joint>

File: forg_description/urdf/wheel.urdf.xacro (robot description, xacro)
@@ -3,5 +3,5 @@
   <xacro:include filename="inertial_macros.urdf.xacro"/>
 	<xacro:arg name="ignition" default="false"/>
-	<xacro:macro name="wheel" params="name parent *origin **mirror">
+	<xacro:macro name="wheel" params="name parent *origin">
     <joint name="${name}_joint" type="continuous">
 			<parent link="${parent}"/>
@@ -14,5 +14,4 @@
 		<link name="${name}_axis">
 			<visual>
-				<xacro:insert_block name="mirror"/>
 				<geometry>
 					<mesh filename="package://forg_description/meshes/wheel_axis.dae"/>
@@ -20,14 +19,9 @@
 			</visual>
 			<collision>
-        <xacro:insert_block name="origin"/>
-        <xacro:insert_block name="mirror"/>
 				<geometry>
 					<mesh filename="package://forg_description/meshes/wheel_axis.dae"/>
 				</geometry>
 			</collision>
-      <xacro:inertial_cylinder mass="0.05" length="0.17" radius="0.00625"> <!-- TODO: replace wheel axis mass with real value -->
-				<xacro:insert_block name="origin"/>
-				<xacro:insert_block name="mirror"/>
-      </xacro:inertial_cylinder>
+      <xacro:inertial_cylinder mass="0.05" length="0.17" radius="0.00625"/> <!-- TODO: replace wheel axis mass with real value -->
 		</link>
     <joint name="${name}_axis_joint" type="fixed">
@@ -39,5 +33,4 @@
 		<link name="${name}">
 			<visual>
-				<xacro:insert_block name="mirror"/>
 				<geometry>
 					<mesh filename="package://forg_description/meshes/wheel.dae"/>
@@ -45,14 +38,9 @@
 			</visual>
 			<collision>
-        <xacro:insert_block name="origin"/>
-        <xacro:insert_block name="mirror"/>
 				<geometry>
 					<mesh filename="package://forg_description/meshes/wheel.dae"/>
 				</geometry>
 			</collision>
-      <xacro:inertial_cylinder mass="0.2" length="0.015" radius="0.06"> <!-- TODO: replace wheel mass with real value -->
-				<xacro:insert_block name="origin"/>
-				<xacro:insert_block name="mirror"/>
-      </xacro:inertial_cylinder>
+      <xacro:inertial_cylinder mass="0.2" length="0.015" radius="0.06"/> <!-- TODO: replace wheel mass with real value -->
 		</link>
 	</xacro:macro>

File: forg_description/urdf/wheel_steering.urdf.xacro (robot description, xacro)
@@ -4,13 +4,12 @@
   <xacro:include filename="wheel.urdf.xacro"/>
 	<xacro:arg name="ignition" default="false"/>
-	<xacro:macro name="wheel_steering" params="name parent *origin **mirror">
+	<xacro:macro name="wheel_steering" params="name parent *origin">
     <joint name="${name}_base_joint" type="fixed">
 			<parent link="${parent}"/>
-			<child link="${name}"/>
+			<child link="${name}_base"/>
       <xacro:insert_block name="origin"/>
 		</joint>
     <link name="${name}_base">
 			<visual>
-				<xacro:insert_block name="mirror"/>
 				<geometry>
 					<mesh filename="package://forg_description/meshes/steering_base.dae"/>
@@ -19,19 +18,32 @@
 			<collision>
         <origin xyz="0 0 0"/>
-        <xacro:insert_block name="mirror"/>
 				<geometry>
 					<mesh filename="package://forg_description/meshes/steering_base.dae"/>
 				</geometry>
 			</collision>
-      <xacro:inertial_box mass="0.05" x="0.17" y="0.00625" z="0.8"> <!-- TODO: replace shoulder axis mass with real value -->
+      <xacro:inertial_box mass="0.05" x="0.17" y="0.00625" z="0.8"/> <!-- TODO: replace shoulder axis mass with real value -->
+		</link>
+    <joint name="${name}_steering_gear_joint" type="continuous">
+			<parent link="${name}_base"/>
+			<child link="${name}_steering_gear"/>
+      <origin xyz="0 0 ${0.15/2 - 0.005/2}"/>
+      <axis xyz="0 0 1"/>
+		</joint>
+    <link name="${name}_steering_gear">
+			<visual>
+				<geometry>
+					<mesh filename="package://forg_description/meshes/steering_gear.dae"/>
+				</geometry>
+			</visual>
+			<collision>
         <origin xyz="0 0 0"/>
-				<xacro:insert_block name="mirror"/>
-      </xacro:inertial_box>
+				<geometry>
+					<mesh filename="package://forg_description/meshes/steering_gear.dae"/>
+				</geometry>
+			</collision>
+      <xacro:inertial_box mass="0.05" x="0.17" y="0.00625" z="0.8"/> <!-- TODO: replace shoulder axis mass with real value -->
 		</link>
-    <xacro:wheel name="${name}" parent="${name}_base">
+  <xacro:wheel name="${name}" parent="${name}_steering_gear">
     <origin xyz="0 ${0.15+0.045+0.11-0.035} ${0.03-0.5}" rpy="${pi/2} 0 ${-pi}"/>
-    <mirror>
-      <origin rpy="0 0 0"/>
-    </mirror>
   </xacro:wheel>
 	</xacro:macro>
