Commit message: configure gazebo ros2 control
it was necessary to erase all semicolons in comments because of a [weird
bug in gazebo_ros2_control
0.4.7](https://github.com/ros-controls/gazebo_ros2_control/issues/295),
I hope it will get fixed soon because I like my "TODO:"s using
folke/todo-comments.nvim

File: forg_description/urdf/base.urdf.xacro (robot description, xacro)
@@ -21,5 +21,5 @@
 				</geometry>
 			</collision>
-      <xacro:inertial_box mass="5" x="0.17" y="0.17" z="0.17"/> <!-- TODO: replace with real values -->
+      <xacro:inertial_box mass="5" x="0.17" y="0.17" z="0.17"/> <!-- TODO replace with real values -->
 		</link>
 	</xacro:macro>

File: forg_description/urdf/forg_bot.urdf.xacro (robot description, xacro)
@@ -1,4 +1,6 @@
-<?xml version="1.0" ?>
+<?xml version="1.0"?>
 <robot xmlns:xacro="http://www.ros.org/wiki/xacro" name="forg_bot">
+	<xacro:arg name="simulation" default="true"/>
   <xacro:include filename="forg_core.urdf.xacro"/>
+  <xacro:include filename="ros2_control.urdf.xacro"/>
 </robot>

File: forg_description/urdf/forg_core.urdf.xacro (robot description, xacro)
@@ -1,3 +1,3 @@
-<?xml version="1.0" ?>
+<?xml version="1.0"?>
 <robot xmlns:xacro="http://www.ros.org/wiki/xacro">
   <xacro:include filename="base.urdf.xacro"/>
@@ -40,5 +40,5 @@
     <mimic joint="shoulder_joint" multiplier="1"/>
     <limit effort="${10}" velocity="${360*2*pi/60}"/>
-    <dynamics damping="0.1" friction="50"/> <!-- TODO: replace with real properties -->
+    <dynamics damping="0.1" friction="50"/> <!-- TODO replace with real properties -->
   </joint>
   <!-- <xacro:mimic_joint_plugin_gazebo name_prefix="shoulder_left" parent_joint="shoulder_joint" mimic_joint="shoulder_left_joint" multiplier="1.0" /> -->
@@ -52,5 +52,5 @@
     <mimic joint="shoulder_joint" multiplier="-1"/>
     <limit effort="${10}" velocity="${360*2*pi/60}"/>
-    <dynamics damping="0.1" friction="50"/> <!-- TODO: replace with real properties -->
+    <dynamics damping="0.1" friction="50"/> <!-- TODO replace with real properties -->
   </joint>
   <xacro:mimic_joint_plugin_gazebo name_prefix="shoulder_right" parent_joint="shoulder_left_joint" mimic_joint="shoulder_right_joint" multiplier="-1.0" debug="false"/>

File: forg_description/urdf/inertial_macros.urdf.xacro (robot description, xacro)
@@ -1,5 +1,5 @@
 <?xml version="1.0"?>
 <robot xmlns:xacro="http://www.ros.org/wiki/xacro" >
-    <!-- Specify some standard inertial calculations https://en.wikipedia.org/wiki/List_of_moments_of_inertia -->
+    <!-- Specify some standard inertial calculations en.wikipedia.org/wiki/List_of_moments_of_inertia -->
     <!-- These make use of xacro's mathematical functionality -->
     <xacro:macro name="inertial_sphere" params="mass radius">

File: forg_description/urdf/left_back_arm.urdf.xacro (robot description, xacro)
@@ -21,5 +21,5 @@
 				</geometry>
 			</collision>
-      <xacro:inertial_box mass="0.05" x="0.17" y="0.00625" z="0.8"/> <!-- TODO: replace shoulder axis mass with real value -->
+      <xacro:inertial_box mass="0.05" x="0.17" y="0.00625" z="0.8"/> <!-- TODO replace shoulder axis mass with real value -->
 		</link>
 	</xacro:macro>

File: forg_description/urdf/left_front_arm.urdf.xacro (robot description, xacro)
@@ -21,5 +21,5 @@
 				</geometry>
 			</collision>
-      <xacro:inertial_box mass="0.05" x="0.17" y="0.00625" z="0.8"/> <!-- TODO: replace shoulder axis mass with real value -->
+      <xacro:inertial_box mass="0.05" x="0.17" y="0.00625" z="0.8"/> <!-- TODO replace shoulder axis mass with real value -->
 		</link>
 	</xacro:macro>

File: forg_description/urdf/left_middle_arm.urdf.xacro (robot description, xacro)
@@ -21,5 +21,5 @@
 				</geometry>
 			</collision>
-      <xacro:inertial_cylinder mass="0.05" length="0.17" radius="0.00625"/> <!-- TODO: replace shoulder axis mass with real value -->
+      <xacro:inertial_cylinder mass="0.05" length="0.17" radius="0.00625"/> <!-- TODO replace shoulder axis mass with real value -->
 		</link>
     <joint name="${name}_joint" type="fixed">
@@ -40,5 +40,5 @@
 				</geometry>
 			</collision>
-      <xacro:inertial_box mass="0.05" x="0.17" y="0.00625" z="0.8"/> <!-- TODO: replace shoulder axis mass with real value -->
+      <xacro:inertial_box mass="0.05" x="0.17" y="0.00625" z="0.8"/> <!-- TODO replace shoulder axis mass with real value -->
 		</link>
 	</xacro:macro>

File: forg_description/urdf/right_back_arm.urdf.xacro (robot description, xacro)
@@ -21,5 +21,5 @@
 				</geometry>
 			</collision>
-      <xacro:inertial_box mass="0.05" x="0.17" y="0.00625" z="0.8"/> <!-- TODO: replace shoulder axis mass with real value -->
+      <xacro:inertial_box mass="0.05" x="0.17" y="0.00625" z="0.8"/> <!-- TODO replace shoulder axis mass with real value -->
 		</link>
 	</xacro:macro>

File: forg_description/urdf/right_front_arm.urdf.xacro (robot description, xacro)
@@ -21,5 +21,5 @@
 				</geometry>
 			</collision>
-      <xacro:inertial_box mass="0.05" x="0.17" y="0.00625" z="0.8"/> <!-- TODO: replace shoulder axis mass with real value -->
+      <xacro:inertial_box mass="0.05" x="0.17" y="0.00625" z="0.8"/> <!-- TODO replace shoulder axis mass with real value -->
 		</link>
 	</xacro:macro>

File: forg_description/urdf/right_middle_arm.urdf.xacro (robot description, xacro)
@@ -21,5 +21,5 @@
 				</geometry>
 			</collision>
-      <xacro:inertial_cylinder mass="0.05" length="0.17" radius="0.00625"/> <!-- TODO: replace shoulder axis mass with real value -->
+      <xacro:inertial_cylinder mass="0.05" length="0.17" radius="0.00625"/> <!-- TODO replace shoulder axis mass with real value -->
 		</link>
     <joint name="${name}_joint" type="fixed">
@@ -40,5 +40,5 @@
 				</geometry>
 			</collision>
-      <xacro:inertial_box mass="0.05" x="0.17" y="0.00625" z="0.8"/> <!-- TODO: replace shoulder axis mass with real value -->
+      <xacro:inertial_box mass="0.05" x="0.17" y="0.00625" z="0.8"/> <!-- TODO replace shoulder axis mass with real value -->
 		</link>
 	</xacro:macro>

File: forg_description/urdf/wheel.urdf.xacro (robot description, xacro)
@@ -9,6 +9,6 @@
 			<xacro:insert_block name="origin"/>
 			<axis xyz="0 0 1"/>
-      <limit effort="${13.3*9.81*2.9}" velocity="${1000*2*pi/60}"/> <!-- TODO: replace with motor limits -->
-			<!--dynamics damping="0.1" friction="1"/--> <!-- TODO: replace with motor + axis properties -->
+      <limit effort="${13.3*9.81*2.9}" velocity="${1000*2*pi/60}"/> <!-- TODO replace with motor limits -->
+			<!--dynamics damping="0.1" friction="1"/--> <!-- TODO replace with motor + axis properties -->
 		</joint>
 		<link name="${name}_axis">
@@ -23,5 +23,5 @@
 				</geometry>
 			</collision>
-      <xacro:inertial_cylinder mass="0.05" length="0.17" radius="0.00625"/> <!-- TODO: replace wheel axis mass with real value -->
+      <xacro:inertial_cylinder mass="0.05" length="0.17" radius="0.00625"/> <!-- TODO replace wheel axis mass with real value -->
 		</link>
     <joint name="${name}_axis_joint" type="fixed">
@@ -42,5 +42,5 @@
 				</geometry>
 			</collision>
-      <xacro:inertial_cylinder mass="0.2" length="0.015" radius="0.06"/> <!-- TODO: replace wheel mass with real value -->
+      <xacro:inertial_cylinder mass="0.2" length="0.015" radius="0.06"/> <!-- TODO replace wheel mass with real value -->
 		</link>
 	</xacro:macro>

File: forg_description/urdf/wheel_steering.urdf.xacro (robot description, xacro)
@@ -21,5 +21,5 @@
 				</geometry>
 			</collision>
-      <xacro:inertial_box mass="0.05" x="0.17" y="0.00625" z="0.8"/> <!-- TODO: replace shoulder axis mass with real value -->
+      <xacro:inertial_box mass="0.05" x="0.17" y="0.00625" z="0.8"/> <!-- TODO replace shoulder axis mass with real value -->
 		</link>
     <joint name="${name}_steering_gear_joint" type="continuous">
@@ -40,5 +40,5 @@
 				</geometry>
 			</collision>
-      <xacro:inertial_box mass="0.05" x="0.17" y="0.00625" z="0.8"/> <!-- TODO: replace shoulder axis mass with real value -->
+      <xacro:inertial_box mass="0.05" x="0.17" y="0.00625" z="0.8"/> <!-- TODO replace shoulder axis mass with real value -->
 		</link>
     <joint name="${name}_steering_joint" type="fixed">
@@ -59,5 +59,5 @@
 				</geometry>
 			</collision>
-      <xacro:inertial_box mass="0.05" x="0.17" y="0.00625" z="0.8"/> <!-- TODO: replace shoulder axis mass with real value -->
+      <xacro:inertial_box mass="0.05" x="0.17" y="0.00625" z="0.8"/> <!-- TODO replace shoulder axis mass with real value -->
 		</link>
   <xacro:wheel name="${name}" parent="${name}_steering">

Commit message: fix wheel track

File: forg_description/urdf/base.urdf.xacro (robot description, xacro)
@@ -15,4 +15,5 @@
 					<mesh filename="package://forg_description/meshes/spine.dae"/>
 				</geometry>
+        <origin rpy="0 0 ${pi/2}"/>
 			</visual>
 			<collision>
@@ -20,4 +21,5 @@
 					<mesh filename="package://forg_description/meshes/spine.dae"/>
 				</geometry>
+        <origin rpy="0 0 ${pi/2}"/>
 			</collision>
       <xacro:inertial_box mass="5" x="0.17" y="0.17" z="0.17"/> <!-- TODO replace with real values -->

File: forg_description/urdf/forg_core.urdf.xacro (robot description, xacro)
@@ -21,5 +21,5 @@
   <link name="base_link"/>
   <xacro:base name="base" parent="base_link">
-    <origin xyz="0 0 0.355" rpy="0 0 ${pi/2}"/> <!-- wheels touch the ground with z=0.345-->
+    <origin xyz="0 0 0.355" rpy="0 0 0"/> <!-- wheels touch the ground with z=0.345-->
   </xacro:base>
   <!-- Add joints and links to simulation differential-like gears -->
@@ -29,5 +29,5 @@
     <parent link="base"/>
     <child link="shoulder_left"/>
-    <origin xyz="${0.255/2 + 0.05} ${0.045-0.225} 0"/>
+    <origin xyz="${-0.045+0.225} ${0.255/2 + 0.05} 0" rpy="0 0 ${pi/2}"/>
     <axis xyz="1 0 0"/>
     <limit effort="${10}" velocity="${360*2*pi/60}"/>
@@ -39,5 +39,5 @@
     <parent link="base"/>
     <child link="shoulder_right"/>
-    <origin xyz="${-0.255/2 - 0.05} ${0.045-0.225} 0"/>
+    <origin xyz="${-0.045+0.225} ${-0.255/2 - 0.05} 0" rpy="0 0 ${pi/2}"/>
     <axis xyz="1 0 0"/>
     <limit effort="${10}" velocity="${360*2*pi/60}"/>
