Commit message: add middle arm

File: forg_description/urdf/forg_core.urdf.xacro (robot description, xacro)
@@ -2,10 +2,37 @@
 <robot xmlns:xacro="http://www.ros.org/wiki/xacro">
   <xacro:include filename="wheel.urdf.xacro"/>
+  <xacro:include filename="base.urdf.xacro"/>
+  <xacro:include filename="middle_arm.urdf.xacro"/>
+  <link name="base_footprint"/>
+  <joint name="base_footprint_to_base_link_joint" type="fixed">
+    <parent link="base_footprint"/>
+    <child link="base_link"/>
+    <origin xyz="0 0 0.5"/>
+    <axis xyz="0 0 1"/>
+  </joint>
   <link name="base_link"/>
-  <xacro:wheel name="front_left_wheel" parent="base_link">
-    <origin xyz="0 0 0.03"/>
+  <xacro:base name="base" parent="base_link">
+    <origin xyz="0 0 0" rpy="0 0 ${pi/2}"/>
+    <mirror>
+      <origin rpy="0 0 0"/>
+    </mirror>
+  </xacro:base>
+  <xacro:middle_arm name="left_middle_arm" parent="base">
+    <origin xyz="${0.255/2 + 0.05} ${0.045-0.225} 0" rpy="0 ${pi/2} 0"/>
+    <mirror>
+      <origin rpy="0 0 0"/>
+    </mirror>
+  </xacro:middle_arm>
+  <xacro:wheel name="front_left_wheel" parent="left_middle_arm">
+    <origin xyz="${0.15+0.045+0.11-0.035} -0.2 ${0.03-0.5}" rpy="0 ${pi/2} 0"/>
     <mirror>
       <origin rpy="0 0 0"/>
     </mirror>
   </xacro:wheel>
+  <xacro:middle_arm name="right_middle_arm" parent="base">
+    <origin xyz="${-0.255/2 - 0.05} ${0.045-0.225} 0" rpy="0 ${pi/2} 0"/>
+    <mirror>
+      <origin rpy="0 0 ${pi}"/>
+    </mirror>
+  </xacro:middle_arm>
 </robot>

File: forg_description/urdf/middle_arm.urdf.xacro (robot description, xacro)
@@ -3,18 +3,17 @@
   <xacro:include filename="inertial_macros.urdf.xacro"/>
 	<xacro:arg name="ignition" default="false"/>
-	<xacro:macro name="wheel" params="name parent *origin **mirror">
-    <joint name="${name}_joint" type="continuous">
+	<xacro:macro name="middle_arm" params="name parent *origin **mirror">
+    <joint name="${name}_shoulder_axis_joint" type="continuous">
 			<parent link="${parent}"/>
-			<child link="${name}_axis"/>
+			<child link="${name}_shoulder_axis"/>
 			<xacro:insert_block name="origin"/>
+      <xacro:insert_block name="mirror"/>
 			<axis xyz="0 0 1"/>
-      <limit effort="${13.3*9.81*2.9}" velocity="${1000*2*pi/60}"/> <!-- TODO: replace with motor limits -->
-			<!--dynamics damping="0.1" friction="1"/--> <!-- TODO: replace with motor + axis properties -->
 		</joint>
-		<link name="${name}_axis">
+    <link name="${name}_shoulder_axis">
 			<visual>
 				<xacro:insert_block name="mirror"/>
 				<geometry>
-					<mesh filename="package://forg_description/meshes/wheel_axis.dae"/>
+					<mesh filename="package://forg_description/meshes/shoulder_axis.dae"/>
 				</geometry>
 			</visual>
@@ -23,23 +22,23 @@
         <xacro:insert_block name="mirror"/>
 				<geometry>
-					<mesh filename="package://forg_description/meshes/wheel_axis.dae"/>
+					<mesh filename="package://forg_description/meshes/shoulder_axis.dae"/>
 				</geometry>
 			</collision>
-      <xacro:inertial_cylinder mass="0.05" length="0.17" radius="0.00625"> <!-- TODO: replace wheel axis mass with real value -->
+      <xacro:inertial_cylinder mass="0.05" length="0.17" radius="0.00625"> <!-- TODO: replace shoulder axis mass with real value -->
 				<xacro:insert_block name="origin"/>
 				<xacro:insert_block name="mirror"/>
       </xacro:inertial_cylinder>
 		</link>
-    <joint name="${name}_axis_joint" type="fixed">
-			<parent link="${name}_axis"/>
+    <joint name="${name}_joint" type="fixed">
+			<parent link="${name}_shoulder_axis"/>
 			<child link="${name}"/>
-      <origin rpy="0 ${-pi/2} 0"/>
-			<axis xyz="1 0 0"/>
+      <origin xyz="0 0 ${-0.005}" rpy="0 ${-pi/2} 0"/>
+			<axis xyz="0 0 1"/>
 		</joint>
-		<link name="${name}">
+    <link name="${name}">
 			<visual>
 				<xacro:insert_block name="mirror"/>
 				<geometry>
-					<mesh filename="package://forg_description/meshes/wheel.dae"/>
+					<mesh filename="package://forg_description/meshes/middle_arm.dae"/>
 				</geometry>
 			</visual>
@@ -48,8 +47,8 @@
         <xacro:insert_block name="mirror"/>
 				<geometry>
-					<mesh filename="package://forg_description/meshes/wheel.dae"/>
+					<mesh filename="package://forg_description/meshes/middle_arm.dae"/>
 				</geometry>
 			</collision>
-      <xacro:inertial_cylinder mass="0.2" length="0.015" radius="0.06"> <!-- TODO: replace wheel mass with real value -->
+      <xacro:inertial_cylinder mass="0.05" length="0.17" radius="0.00625"> <!-- TODO: replace shoulder axis mass with real value -->
 				<xacro:insert_block name="origin"/>
 				<xacro:insert_block name="mirror"/>

Commit message: add wheels to the rest of the urdf

File: forg_description/urdf/forg_core.urdf.xacro (robot description, xacro)
@@ -33,4 +33,10 @@
     <origin xyz="${0.045/2 + 0.11 - 0.07/2} ${0.18 + 0.2} ${-0.075}" rpy="0 0 0"/>
   </xacro:left_back_arm>
+  <xacro:wheel_steering name="left_middle_wheel" parent="left_back_arm">
+    <origin xyz="0 ${-0.045 - 0.1 - 0.14/2} ${-0.075}" rpy="${pi} 0 0"/>
+  </xacro:wheel_steering>
+  <xacro:wheel_steering name="left_back_wheel" parent="left_back_arm">
+    <origin xyz="0 ${0.045 + 0.1 + 0.14/2} ${-0.075}" rpy="${pi} 0 0"/>
+  </xacro:wheel_steering>
   <xacro:right_middle_arm name="right_middle_arm" parent="base">
     <origin xyz="${-0.255/2 - 0.05} ${0.045-0.225} 0" rpy="0 ${pi/2} 0"/>
@@ -39,4 +45,13 @@
     <origin xyz="${-0.045/2 - 0.11 + 0.07/2} 0 0" rpy="0 0 0"/>
   </xacro:right_front_arm>
+  <xacro:wheel_steering name="right_front_wheel" parent="right_front_arm">
+    <origin xyz="0 ${-0.07-0.18-0.015} ${-0.15}" rpy="${pi} 0 0"/>
+  </xacro:wheel_steering>
+  <xacro:wheel_steering name="right_middle_wheel" parent="right_back_arm">
+    <origin xyz="0 ${-0.045 - 0.1 - 0.14/2} ${-0.075}" rpy="${pi} 0 0"/>
+  </xacro:wheel_steering>
+  <xacro:wheel_steering name="right_back_wheel" parent="right_back_arm">
+    <origin xyz="0 ${0.045 + 0.1 + 0.14/2} ${-0.075}" rpy="${pi} 0 0"/>
+  </xacro:wheel_steering>
   <xacro:right_back_arm name="right_back_arm" parent="right_middle_arm">
     <origin xyz="${-0.045/2 - 0.11 + 0.07/2} ${0.18 + 0.2} ${-0.075}" rpy="0 0 0"/>

File: forg_description/urdf/wheel_steering.urdf.xacro (robot description, xacro)
@@ -17,5 +17,4 @@
 			</visual>
 			<collision>
-        <origin xyz="0 0 0"/>
 				<geometry>
 					<mesh filename="package://forg_description/meshes/steering_base.dae"/>
@@ -27,5 +26,5 @@
 			<parent link="${name}_base"/>
 			<child link="${name}_steering_gear"/>
-      <origin xyz="0 0 ${0.15/2 - 0.005/2}"/>
+      <origin xyz="0 0 ${0.15/2 - 0.005}"/>
       <axis xyz="0 0 1"/>
 		</joint>
@@ -37,5 +36,4 @@
 			</visual>
 			<collision>
-        <origin xyz="0 0 0"/>
 				<geometry>
 					<mesh filename="package://forg_description/meshes/steering_gear.dae"/>
@@ -44,6 +42,25 @@
       <xacro:inertial_box mass="0.05" x="0.17" y="0.00625" z="0.8"/> <!-- TODO: replace shoulder axis mass with real value -->
 		</link>
-  <xacro:wheel name="${name}" parent="${name}_steering_gear">
-    <origin xyz="0 ${0.15+0.045+0.11-0.035} ${0.03-0.5}" rpy="${pi/2} 0 ${-pi}"/>
+    <joint name="${name}_steering_joint" type="fixed">
+			<parent link="${name}_steering_gear"/>
+			<child link="${name}_steering"/>
+      <origin xyz="0 0 ${0.06 + 0.005}" rpy="-${pi/2} 0 0"/>
+      <axis xyz="0 0 1"/>
+		</joint>
+    <link name="${name}_steering">
+			<visual>
+				<geometry>
+					<mesh filename="package://forg_description/meshes/wheel_steering.dae"/>
+				</geometry>
+			</visual>
+			<collision>
+				<geometry>
+					<mesh filename="package://forg_description/meshes/wheel_steering.dae"/>
+				</geometry>
+			</collision>
+      <xacro:inertial_box mass="0.05" x="0.17" y="0.00625" z="0.8"/> <!-- TODO: replace shoulder axis mass with real value -->
+		</link>
+  <xacro:wheel name="${name}" parent="${name}_steering">
+      <origin rpy="0 ${pi/2} 0"/>
   </xacro:wheel>
 	</xacro:macro>

Commit message: Add joints and links to simulation differential-like gears
This is made in order to make the rotation of the shoulders to be the
oposite to one another

File: forg_description/urdf/forg_core.urdf.xacro (robot description, xacro)
@@ -15,5 +15,5 @@
     <child link="base_link"/>
     <origin xyz="0 0 0.5"/>
-    <axis xyz="0 0 1"/>
+    <axis xyz="1 0 0"/>
   </joint>
   <link name="base_link"/>
@@ -21,6 +21,35 @@
     <origin xyz="0 0 0.5" rpy="0 0 ${pi/2}"/>
   </xacro:base>
-  <xacro:left_middle_arm name="left_middle_arm" parent="base">
-    <origin xyz="${0.255/2 + 0.05} ${0.045-0.225} 0" rpy="0 ${pi/2} 0"/>
+  <!-- Add joints and links to simulation differential-like gears -->
+  <!-- This is made in order to make the rotation of the shoulders to be the oposite to one another-->
+  <joint name="shoulder_joint" type="continuous">
+    <parent link="base"/>
+    <child link="shoulder"/>
+    <origin xyz="0 ${-0.225} 0"/>
+    <axis xyz="0 1 0"/>
+  </joint>
+  <link name="shoulder">
+  </link>
+  <joint name="shoulder_left_joint" type="continuous">
+    <parent link="base"/>
+    <child link="shoulder_left"/>
+    <origin xyz="${0.255/2 + 0.05} ${0.045-0.225} 0"/>
+    <axis xyz="1 0 0"/>
+    <mimic joint="shoulder_joint" multiplier="1"/>
+  </joint>
+  <link name="shoulder_left">
+  </link>
+  <joint name="shoulder_right_joint" type="continuous">
+    <parent link="base"/>
+    <child link="shoulder_right"/>
+    <origin xyz="${-0.255/2 - 0.05} ${0.045-0.225} 0"/>
+    <axis xyz="1 0 0"/>
+    <mimic joint="shoulder_joint" multiplier="-1"/>
+  </joint>
+  <link name="shoulder_right">
+  </link>
+  <!-- End of differential-like gears -->
+  <xacro:left_middle_arm name="left_middle_arm" parent="shoulder_left">
+    <origin xyz="0 0 0" rpy="0 ${pi/2} 0"/>
   </xacro:left_middle_arm>
   <xacro:left_front_arm name="left_front_arm" parent="left_middle_arm">
@@ -39,6 +68,6 @@
     <origin xyz="0 ${0.045 + 0.1 + 0.14/2} ${-0.075}" rpy="${pi} 0 0"/>
   </xacro:wheel_steering>
-  <xacro:right_middle_arm name="right_middle_arm" parent="base">
-    <origin xyz="${-0.255/2 - 0.05} ${0.045-0.225} 0" rpy="0 ${pi/2} 0"/>
+  <xacro:right_middle_arm name="right_middle_arm" parent="shoulder_right">
+    <origin xyz="0 0 0" rpy="0 ${pi/2} 0"/>
   </xacro:right_middle_arm>
   <xacro:right_front_arm name="right_front_arm" parent="right_middle_arm">

File: forg_description/urdf/left_middle_arm.urdf.xacro (robot description, xacro)
@@ -4,5 +4,5 @@
 	<xacro:arg name="ignition" default="false"/>
 	<xacro:macro name="left_middle_arm" params="name parent *origin">
-    <joint name="${name}_shoulder_axis_joint" type="continuous">
+    <joint name="${name}_shoulder_axis_joint" type="fixed">
 			<parent link="${parent}"/>
 			<child link="${name}_shoulder_axis"/>

File: forg_description/urdf/right_middle_arm.urdf.xacro (robot description, xacro)
@@ -4,5 +4,5 @@
 	<xacro:arg name="ignition" default="false"/>
 	<xacro:macro name="right_middle_arm" params="name parent *origin">
-    <joint name="${name}_shoulder_axis_joint" type="continuous">
+    <joint name="${name}_shoulder_axis_joint" type="fixed">
 			<parent link="${parent}"/>
 			<child link="${name}_shoulder_axis"/>

Commit message: remove base_footprint in urdf

File: forg_description/urdf/forg_core.urdf.xacro (robot description, xacro)
@@ -10,14 +10,7 @@
   <xacro:include filename="wheel_steering.urdf.xacro"/>
   <xacro:include filename="wheel.urdf.xacro"/>
-  <link name="base_footprint"/>
-  <joint name="base_footprint_to_base_link_joint" type="fixed">
-    <parent link="base_footprint"/>
-    <child link="base_link"/>
-    <origin xyz="0 0 0.5"/>
-    <axis xyz="1 0 0"/>
-  </joint>
   <link name="base_link"/>
   <xacro:base name="base" parent="base_link">
-    <origin xyz="0 0 0.5" rpy="0 0 ${pi/2}"/>
+    <origin xyz="0 0 0.355" rpy="0 0 ${pi/2}"/> <!-- wheels touch the ground with z=0.345-->
   </xacro:base>
   <!-- Add joints and links to simulation differential-like gears -->

Commit message: integrate mimic_joint_plugin into the simulation

File: forg_description/urdf/forg_core.urdf.xacro (robot description, xacro)
@@ -5,4 +5,5 @@
   <xacro:include filename="left_front_arm.urdf.xacro"/>
   <xacro:include filename="left_back_arm.urdf.xacro"/>
+  <xacro:include filename="mimic_joint_plugin_macro.urdf.xacro"/>
   <xacro:include filename="right_middle_arm.urdf.xacro"/>
   <xacro:include filename="right_front_arm.urdf.xacro"/>
@@ -10,4 +11,12 @@
   <xacro:include filename="wheel_steering.urdf.xacro"/>
   <xacro:include filename="wheel.urdf.xacro"/>
+  <!-- <link name="world"> -->
+  <!-- </link> -->
+  <!---->
+  <!-- <joint name="world_joint" type="fixed"> -->
+  <!--   <parent link="world"/> -->
+  <!--   <child link="base_link"/> -->
+  <!--   <origin xyz="0 0 0.01"/> -->
+  <!-- </joint> -->
   <link name="base_link"/>
   <xacro:base name="base" parent="base_link">
@@ -30,5 +39,8 @@
     <axis xyz="1 0 0"/>
     <mimic joint="shoulder_joint" multiplier="1"/>
+    <limit effort="${10}" velocity="${360*2*pi/60}"/>
+    <dynamics damping="0.1" friction="50"/> <!-- TODO: replace with real properties -->
   </joint>
+  <!-- <xacro:mimic_joint_plugin_gazebo name_prefix="shoulder_left" parent_joint="shoulder_joint" mimic_joint="shoulder_left_joint" multiplier="1.0" /> -->
   <link name="shoulder_left">
   </link>
@@ -39,5 +51,8 @@
     <axis xyz="1 0 0"/>
     <mimic joint="shoulder_joint" multiplier="-1"/>
+    <limit effort="${10}" velocity="${360*2*pi/60}"/>
+    <dynamics damping="0.1" friction="50"/> <!-- TODO: replace with real properties -->
   </joint>
+  <xacro:mimic_joint_plugin_gazebo name_prefix="shoulder_right" parent_joint="shoulder_left_joint" mimic_joint="shoulder_right_joint" multiplier="-1.0" debug="false"/>
   <link name="shoulder_right">
   </link>

Commit message: implement inverse kinematics for holonomic_rover_controller

File: forg_description/urdf/forg_core.urdf.xacro (robot description, xacro)
@@ -54,5 +54,5 @@
     <dynamics damping="0.1" friction="50"/> <!-- TODO replace with real properties -->
   </joint>
-  <xacro:mimic_joint_plugin_gazebo name_prefix="shoulder_right" parent_joint="shoulder_left_joint" mimic_joint="shoulder_right_joint" multiplier="-1.0" debug="false"/>
+  <!-- <xacro:mimic_joint_plugin_gazebo name_prefix="shoulder_right" parent_joint="shoulder_left_joint" mimic_joint="shoulder_right_joint" multiplier="-1.0" debug="false"/> -->
   <link name="shoulder_right">
   </link>

File: forg_description/urdf/left_front_arm.urdf.xacro (robot description, xacro)
@@ -4,9 +4,8 @@
 	<xacro:arg name="ignition" default="false"/>
 	<xacro:macro name="left_front_arm" params="name parent *origin">
-    <joint name="${name}_joint" type="continuous">
+    <joint name="${name}_joint" type="fixed">
 			<parent link="${parent}"/>
 			<child link="${name}"/>
       <xacro:insert_block name="origin"/>
-			<axis xyz="1 0 0"/>
 		</joint>
     <link name="${name}">

File: forg_description/urdf/right_front_arm.urdf.xacro (robot description, xacro)
@@ -4,9 +4,8 @@
 	<xacro:arg name="ignition" default="false"/>
 	<xacro:macro name="right_front_arm" params="name parent *origin">
-    <joint name="${name}_joint" type="continuous">
+    <joint name="${name}_joint" type="fixed">
 			<parent link="${parent}"/>
 			<child link="${name}"/>
       <xacro:insert_block name="origin"/>
-			<axis xyz="1 0 0"/>
 		</joint>
     <link name="${name}">

File: forg_description/urdf/ros2_control.urdf.xacro (robot description, xacro)
@@ -79,4 +79,18 @@
         <state_interface name="effort"/>
       </joint>
+      <joint name="shoulder_left_joint">
+        <command_interface name="position"/>
+        <state_interface name="position"/>
+        <state_interface name="velocity"/>
+        <state_interface name="effort"/>
+      </joint>
+      <joint name="shoulder_right_joint">
+        <param name="mimic">shoulder_left_joint</param>
+        <param name="multiplier">-1</param>
+        <command_interface name="position"/>
+        <state_interface name="position"/>
+        <state_interface name="velocity"/>
+        <state_interface name="effort"/>
+      </joint>
     </ros2_control>
     <gazebo>

File: forg_description/urdf/wheel.urdf.xacro (robot description, xacro)
@@ -10,5 +10,6 @@
 			<axis xyz="0 0 1"/>
       <limit effort="${13.3*9.81*2.9}" velocity="${1000*2*pi/60}"/> <!-- TODO replace with motor limits -->
-			<!--dynamics damping="0.1" friction="1"/--> <!-- TODO replace with motor + axis properties -->
+      <!-- <dynamics damping="0.1" friction="1"/> -->
+      <!-- TODO replace with motor + axis properties-->
 		</joint>
 		<link name="${name}_axis">

Commit message: add PID using gazebo::physics::JointController in mimic_joint_plugin_gazebo

File: forg_description/urdf/forg_core.urdf.xacro (robot description, xacro)
@@ -54,5 +54,5 @@
     <dynamics damping="0.1" friction="50"/> <!-- TODO replace with real properties -->
   </joint>
-  <!-- <xacro:mimic_joint_plugin_gazebo name_prefix="shoulder_right" parent_joint="shoulder_left_joint" mimic_joint="shoulder_right_joint" multiplier="-1.0" debug="false"/> -->
+  <xacro:mimic_joint_plugin_gazebo name_prefix="shoulder_right" parent_joint="shoulder_left_joint" mimic_joint="shoulder_right_joint" multiplier="-1.0" debug="false" use_pid="true" kp="100.0" ki="100.0" kd="100.0"/>
   <link name="shoulder_right">
   </link>

File: forg_description/urdf/ros2_control.urdf.xacro (robot description, xacro)
@@ -79,18 +79,18 @@
         <state_interface name="effort"/>
       </joint>
-      <joint name="shoulder_left_joint">
-        <command_interface name="position"/>
-        <state_interface name="position"/>
-        <state_interface name="velocity"/>
-        <state_interface name="effort"/>
-      </joint>
-      <joint name="shoulder_right_joint">
-        <param name="mimic">shoulder_left_joint</param>
-        <param name="multiplier">-1</param>
-        <command_interface name="position"/>
-        <state_interface name="position"/>
-        <state_interface name="velocity"/>
-        <state_interface name="effort"/>
-      </joint>
+      <!-- <joint name="shoulder_left_joint"> -->
+      <!--   <command_interface name="position"/> -->
+      <!--   <state_interface name="position"/> -->
+      <!--   <state_interface name="velocity"/> -->
+      <!--   <state_interface name="effort"/> -->
+      <!-- </joint> -->
+      <!-- <joint name="shoulder_right_joint"> -->
+      <!--   <param name="mimic">shoulder_left_joint</param> -->
+      <!--   <param name="multiplier">-1</param> -->
+      <!--   <command_interface name="position"/> -->
+      <!--   <state_interface name="position"/> -->
+      <!--   <state_interface name="velocity"/> -->
+      <!--   <state_interface name="effort"/> -->
+      <!-- </joint> -->
     </ros2_control>
     <gazebo>

Commit message: separate run and enter recipes

File: forg_description/urdf/forg_core.urdf.xacro (robot description, xacro)
@@ -5,4 +5,5 @@
   <xacro:include filename="left_front_arm.urdf.xacro"/>
   <xacro:include filename="left_back_arm.urdf.xacro"/>
+  <xacro:include filename="lidar.urdf.xacro"/>
   <xacro:include filename="right_middle_arm.urdf.xacro"/>
   <xacro:include filename="right_front_arm.urdf.xacro"/>
@@ -90,3 +91,6 @@
     <origin xyz="${-0.045/2 - 0.11 + 0.07/2} ${0.18 + 0.2} ${-0.075}" rpy="0 0 0"/>
   </xacro:right_back_arm>
+  <xacro:lidar name="lidar" parent="base">
+    <origin xyz="0 0 0.2" rpy="0 0 0"/>
+  </xacro:lidar>
 </robot>

File: forg_description/urdf/lidar.urdf.xacro (robot description, xacro)
@@ -1,4 +1,5 @@
 <?xml version="1.0"?>
 <robot xmlns:xacro="http://www.ros.org/wiki/xacro" >
+  <xacro:include filename="inertial_macros.urdf.xacro"/>
 	<xacro:macro name="lidar" params="name parent scan_topic:=scan *origin">
     <joint name="${name}_joint" type="fixed">
@@ -26,7 +27,5 @@
         </geometry>
       </collision>
-      <xacro:inertial_cylinder mass="0.1" length="0.04" radius="0.05">
-        <origin xyz="0 0 0" rpy="0 0 0"/>
-      </xacro:inertial_cylinder>
+      <xacro:inertial_cylinder mass="0.1" length="0.04" radius="0.05"/>
     </link>
     <gazebo reference="${name}">

Commit message: wip

File: forg_description/urdf/forg_core.urdf.xacro (robot description, xacro)
@@ -25,12 +25,4 @@
   <!-- Add joints and links to simulation differential-like gears -->
   <!-- This is made in order to make the rotation of the shoulders to be the oposite to one another-->
-  <joint name="shoulder_joint" type="continuous">
-    <parent link="base"/>
-    <child link="shoulder"/>
-    <origin xyz="0 ${-0.225} 0"/>
-    <axis xyz="0 1 0"/>
-  </joint>
-  <link name="shoulder">
-  </link>
   <joint name="shoulder_left_joint" type="continuous">
     <mimic joint="shoulder_right_joint" multiplier="-1"/>

Commit message: undo debug

File: forg_description/urdf/forg_core.urdf.xacro (robot description, xacro)
@@ -17,5 +17,5 @@
   <!--   <parent link="world"/> -->
   <!--   <child link="base_link"/> -->
-  <!--   <origin xyz="0 0 0.01"/> -->
+  <!--   <origin xyz="0 0 0.5"/> -->
   <!-- </joint> -->
   <link name="base_link"/>

Commit message: fix contact problems

File: forg_description/urdf/forg_core.urdf.xacro (robot description, xacro)
@@ -26,5 +26,4 @@
   <!-- This is made in order to make the rotation of the shoulders to be the oposite to one another-->
   <joint name="shoulder_left_joint" type="continuous">
-    <mimic joint="shoulder_right_joint" multiplier="-1"/>
     <parent link="base"/>
     <child link="shoulder_left"/>
@@ -32,5 +31,5 @@
     <axis xyz="1 0 0"/>
     <limit effort="${10}" velocity="${360*2*pi/60}"/>
-    <dynamics damping="0.1" friction="50"/> <!-- TODO replace with real properties -->
+    <dynamics damping="0.1" friction="0.0"/>
   </joint>
   <link name="shoulder_left">
@@ -42,5 +41,5 @@
     <axis xyz="1 0 0"/>
     <limit effort="${10}" velocity="${360*2*pi/60}"/>
-    <dynamics damping="0.1" friction="50"/> <!-- TODO replace with real properties -->
+    <dynamics damping="0.1" friction="0.0"/>
   </joint>
   <link name="shoulder_right">

File: forg_description/urdf/wheel.urdf.xacro (robot description, xacro)
@@ -39,6 +39,6 @@
 			<collision>
 				<geometry>
-					<!-- <mesh filename="package://forg_description/meshes/wheel.dae"/> -->
-          <sphere radius="0.06"/>
+					<mesh filename="package://forg_description/meshes/wheel.dae"/>
+          <!-- <sphere radius="0.06"/> -->
 				</geometry>
 			</collision>
