Commit message: change navigation config

File: forg_description/urdf/forg_core.urdf.xacro (robot description, xacro)
@@ -26,4 +26,5 @@
   <!-- This is made in order to make the rotation of the shoulders to be the oposite to one another-->
   <joint name="shoulder_left_joint" type="continuous">
+    <mimic joint="shoulder_right_joint" multiplier="-1"/>
     <parent link="base"/>
     <child link="shoulder_left"/>
@@ -31,5 +32,5 @@
     <axis xyz="1 0 0"/>
     <limit effort="${10}" velocity="${360*2*pi/60}"/>
-    <dynamics damping="0.1" friction="0.0"/>
+    <dynamics damping="0.1" friction="50"/> <!-- TODO replace with real properties -->
   </joint>
   <link name="shoulder_left">
@@ -41,5 +42,5 @@
     <axis xyz="1 0 0"/>
     <limit effort="${10}" velocity="${360*2*pi/60}"/>
-    <dynamics damping="0.1" friction="0.0"/>
+    <dynamics damping="0.1" friction="50"/> <!-- TODO replace with real properties -->
   </joint>
   <link name="shoulder_right">
